Commit message: complete ROS 2 navigation assignment deliverables

File: testbed_description/urdf/materials.xacro (robot description, xacro)
@@ -4,3 +4,18 @@
   <color rgba="0.700 0.700 0.700 1.000"/>
 </material>
+<material name="chassis_gray">
+  <color rgba="0.200 0.200 0.200 1.000"/>
+</material>
+<material name="wheel_black">
+  <color rgba="0.050 0.050 0.050 1.000"/>
+</material>
+<material name="caster_dark">
+  <color rgba="0.100 0.100 0.100 1.000"/>
+</material>
+<material name="lidar_blue">
+  <color rgba="0.100 0.400 0.900 1.000"/>
+</material>
+<material name="imu_red">
+  <color rgba="0.900 0.100 0.100 1.000"/>
+</material>
 </robot>

File: testbed_description/urdf/testbed.xacro (robot description, xacro)
@@ -23,5 +23,5 @@
       <mesh filename="file://$(find testbed_description)/meshes/base_link.stl" scale="0.001 0.001 0.001"/>
     </geometry>
-    <material name="silver"/>
+    <material name="chassis_gray"/>
   </visual>
   <collision>
@@ -43,5 +43,5 @@
       <mesh filename="file://$(find testbed_description)/meshes/left_wheel_1.stl" scale="0.001 0.001 0.001"/>
     </geometry>
-    <material name="silver"/>
+    <material name="wheel_black"/>
   </visual>
   <collision>
@@ -63,5 +63,5 @@
       <mesh filename="file://$(find testbed_description)/meshes/caster_1.stl" scale="0.001 0.001 0.001"/>
     </geometry>
-    <material name="silver"/>
+    <material name="caster_dark"/>
   </visual>
   <collision>
@@ -83,5 +83,5 @@
       <mesh filename="file://$(find testbed_description)/meshes/caster_2.stl" scale="0.001 0.001 0.001"/>
     </geometry>
-    <material name="silver"/>
+    <material name="caster_dark"/>
   </visual>
   <collision>
@@ -103,5 +103,5 @@
       <mesh filename="file://$(find testbed_description)/meshes/caster_3.stl" scale="0.001 0.001 0.001"/>
     </geometry>
-    <material name="silver"/>
+    <material name="caster_dark"/>
   </visual>
   <collision>
@@ -123,5 +123,5 @@
       <mesh filename="file://$(find testbed_description)/meshes/caster_4.stl" scale="0.001 0.001 0.001"/>
     </geometry>
-    <material name="silver"/>
+    <material name="caster_dark"/>
   </visual>
   <collision>
@@ -143,5 +143,5 @@
       <mesh filename="file://$(find testbed_description)/meshes/lidar_link_1.stl" scale="0.001 0.001 0.001"/>
     </geometry>
-    <material name="silver"/>
+    <material name="lidar_blue"/>
   </visual>
   <collision>
@@ -163,5 +163,5 @@
       <mesh filename="file://$(find testbed_description)/meshes/imu_link_1.stl" scale="0.001 0.001 0.001"/>
     </geometry>
-    <material name="silver"/>
+    <material name="imu_red"/>
   </visual>
   <collision>
@@ -203,5 +203,5 @@
       <mesh filename="file://$(find testbed_description)/meshes/right_wheel_1.stl" scale="0.001 0.001 0.001"/>
     </geometry>
-    <material name="silver"/>
+    <material name="wheel_black"/>
   </visual>
   <collision>
